File: pcb/CZTKeyRev0.sch (KiCad schematic (older format))
At the start: 269 parts, among them U1 proton_c

Commit message: Generated gerber, added silkscreen and more
Parts:
- removed R5: 10K, Resistor_SMD:R_0603_1608Metric, symbol Device:R_Small
- added C10, C11, C12, C13, C14, C15, C16, C17, C18, C19, C20, C21, C22, C23, C24, C25, C26, C27, C28, C29, C3, C30, C31, C32, C33, C34, C35, C36, C37, C38, C39, C4, C40, C41, C42, C43, C44, C45, C46, C47, C5, C6, C7, C8, C9: 100n, decoup cap:CAPC2012X70, symbol Device:C_Small
- added D87: D_Small, Diode_THT:D_DO-35_SOD27_P5.08mm_Vertical_KathodeUp, symbol Device:D_Small
Connections:
- net labels added: ENC_S1, ENC_S2
- wire segments 556 -> 593
- no-connect marks 1 -> 0
Other:
- note added: "decoupling capacitory - smd C49678"
- moved on the sheet: WS77, WS87

Commit message: batchcommit
Parts:
- removed C10, C11, C12, C13, C14, C15, C16, C17, C18, C19, C20, C21, C22, C23, C24, C25, C26, C27, C28, C29, C3, C30, C31, C32, C33, C34, C35, C36, C37, C38, C39, C4, C40, C41, C42, C43, C44, C45, C46, C47, C5, C6, C7, C8, C9: 100n, decoup cap:CAPC2012X70, symbol Device:C_Small
- removed WS1, WS10, WS11, WS12, WS13, WS14, WS15, WS2, WS3, WS31, WS4, WS47, WS5, WS6, WS62, WS7, WS77, WS8, WS9: WS2812B, WS2812B-edited:Neopixel_easy_LED_WS2812B_PLCC4_5.0x5.0mm_P3.2mm, symbol LED:WS2812B
Connections:
- net D_ROW3: now also WS32.4 (DIN)
- net D_ROW4: now also WS48.4 (DIN)
- net D_ROW5: now also WS63.4 (DIN)
- net D_ROW6: now also WS78.4 (DIN)
- net RGB_MATRIX: now also WS16.4 (DIN)
Other:
- moved on the sheet: WS16, WS17, WS18, WS19, WS20, WS21, WS22, WS23, WS24, WS25, WS26, WS27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

Commit message: added mounting pads
Parts:
- added PCB_BC, PCB_BL, PCB_BR, PCB_TC, PCB_TL, PCB_TR, PLATE_BC, PLATE_BL, PLATE_BR, PLATE_TC, PLATE_TL, PLATE_TR: MountingHole_Pad, symbol Mechanical:MountingHole_Pad
Other:
- moved on the sheet: WS16, WS17, WS18, WS19, WS20, WS21, WS22, WS23, WS24, WS25, WS26, WS27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
