File: pcb/_autosave-CZTKeyRev0.sch (KiCad schematic (older format))
At the start: 195 parts, among them U1 proton_c

Commit message: sync
Parts:
- added BJ_LED5V: Barrel_Jack, symbol Connector:Barrel_Jack
- added D?: SK6812MINI, LED_SMD:LED_SK6812MINI_PLCC4_3.5x3.5mm_P1.75mm, symbol LED:SK6812MINI
Connections:
- net RGB_MATRIX: now also D?.3 (DIN)
- new net EXT_5V: BJ_LED5V.1
- new net EXT_GND: BJ_LED5V.2
- no-connect marks 0 -> 1
Other:
- moved on the sheet: D?
Changed lines of the file:
@@
 L LED:SK6812MINI D?
 U 1 1 5FCBCA87
-P 2650 11550
-F 0 "D?" H 2994 11596 50  0000 L CNN
-F 1 "SK6812MINI" H 2994 11505 50  0000 L CNN
-F 2 "LED_SMD:LED_SK6812MINI_PLCC4_3.5x3.5mm_P1.75mm" H 2700 11250 50  0001 L TNN
-F 3 "https://cdn-shop.adafruit.com/product-files/2686/SK6812MINI_REV.01-1-2.pdf" H 2750 11175 50  0001 L TNN
-	1    2650 11550
+P 3050 11100
+F 0 "D?" H 3394 11146 50  0000 L CNN
+F 1 "SK6812MINI" H 3394 11055 50  0000 L CNN
+F 2 "LED_SMD:LED_SK6812MINI_PLCC4_3.5x3.5mm_P1.75mm" H 3100 10800 50  0001 L TNN
+F 3 "https://cdn-shop.adafruit.com/product-files/2686/SK6812MINI_REV.01-1-2.pdf" H 3150 10725 50  0001 L TNN
+	1    3050 11100
 	1    0    0    -1
 $EndComp
+$Comp
+L Connector:Barrel_Jack BJ_LED5V
+U 1 1 5FC7DC4D
+P 1850 10150
+F 0 "BJ_LED5V" H 1907 10475 50  0000 C CNN
+F 1 "Barrel_Jack" H 1907 10384 50  0000 C CNN
+F 2 "" H 1900 10110 50  0001 C CNN
+F 3 "~" H 1900 10110 50  0001 C CNN
+	1    1850 10150
+	1    0    0    -1
+$EndComp
+Text GLabel 2750 11100 0    50   Input ~ 0
+RGB_MATRIX
+$Comp
+L LED:SK6812MINI D?
+U 1 1 5FC81A59
+P 4050 11100
+F 0 "D?" H 4394 11146 50  0000 L CNN
+F 1 "SK6812MINI" H 4394 11055 50  0000 L CNN
+F 2 "LED_SMD:LED_SK6812MINI_PLCC4_3.5x3.5mm_P1.75mm" H 4100 10800 50  0001 L TNN
+F 3 "https://cdn-shop.adafruit.com/product-files/2686/SK6812MINI_REV.01-1-2.pdf" H 4150 10725 50  0001 L TNN
+	1    4050 11100
+	1    0    0    -1
+$EndComp
+NoConn ~ 4350 11100
+Text GLabel 2150 10050 2    50   Input ~ 0
+EXT_5V
+Text GLabel 2150 10250 2    50   Input ~ 0
+EXT_GND
 $EndSCHEMATC
