File: pcb/CZTKeyRev0.kicad_pcb (KiCad board)
At the start: 2 copper layers, 343 x 159 mm, 280 parts, among them U1 proton_c

Commit message: Generated gerber, added silkscreen and more
Parts:
- removed R5: 10K, Resistor_SMD:R_0603_1608Metric
- removed REF** (x11): MountingHole_2.2mm_M2_Pad, MountingHole:MountingHole_2.2mm_M2_Pad
- added C10: 100n, decoup cap:CAPC2012X70, F.Cu at (52.7, 97.8)
- added C11: 100n, decoup cap:CAPC2012X70, F.Cu at (90.8, 97.7)
- added C12: 100n, decoup cap:CAPC2012X70, F.Cu at (128.9, 98.2)
- added C13: 100n, decoup cap:CAPC2012X70, F.Cu at (167.0, 97.5)
- added C14: 100n, decoup cap:CAPC2012X70, F.Cu at (205.1, 98.9)
- added C15: 100n, decoup cap:CAPC2012X70, F.Cu at (243.2, 97.8)
- added C16: 100n, decoup cap:CAPC2012X70, F.Cu at (290.8, 99.8)
- added C17: 100n, decoup cap:CAPC2012X70, F.Cu at (9.78, 97.8)
- added C18: 100n, decoup cap:CAPC2012X70, F.Cu at (62.2, 116.8)
- added C19: 100n, decoup cap:CAPC2012X70, F.Cu at (100.3, 117.1)
- added C20: 100n, decoup cap:CAPC2012X70, F.Cu at (138.4, 117.6)
- added C21: 100n, decoup cap:CAPC2012X70, F.Cu at (176.5, 116.6)
- added C22: 100n, decoup cap:CAPC2012X70, F.Cu at (195.6, 117.7)
- added C23: 100n, decoup cap:CAPC2012X70, F.Cu at (252.9, 116.7)
- added C24: 100n, decoup cap:CAPC2012X70, F.Cu at (295.7, 118.0)
- added C25: 100n, decoup cap:CAPC2012X70, F.Cu at (9.91, 116.6)
- added C26: 100n, decoup cap:CAPC2012X70, F.Cu at (66.9, 136.7)
- added C27: 100n, decoup cap:CAPC2012X70, F.Cu at (105.2, 136.7)
- added C28: 100n, decoup cap:CAPC2012X70, F.Cu at (143.3, 136.4)
- added C29: 100n, decoup cap:CAPC2012X70, F.Cu at (181.2, 136.9)
- added C3: 100n, decoup cap:CAPC2012X70, F.Cu at (76.5, 74.8)
- added C30: 100n, decoup cap:CAPC2012X70, F.Cu at (219.5, 135.8)
- added C31: 100n, decoup cap:CAPC2012X70, F.Cu at (257.7, 136.0)
- added C32: 100n, decoup cap:CAPC2012X70, F.Cu at (333.6, 135.4)
- added C33: 100n, decoup cap:CAPC2012X70, F.Cu at (9.91, 136.9)
- added C34: 100n, decoup cap:CAPC2012X70, F.Cu at (45.7, 156.7)
- added C35: 100n, decoup cap:CAPC2012X70, F.Cu at (95.5, 156.0)
- added C36: 100n, decoup cap:CAPC2012X70, F.Cu at (152.8, 154.8)
- added C37: 100n, decoup cap:CAPC2012X70, F.Cu at (190.6, 155.6)
- added C38: 100n, decoup cap:CAPC2012X70, F.Cu at (228.7, 155.1)
- added C39: 100n, decoup cap:CAPC2012X70, F.Cu at (274.4, 154.9)
- added C4: 100n, decoup cap:CAPC2012X70, F.Cu at (114.6, 74.2)
- added C40: 100n, decoup cap:CAPC2012X70, F.Cu at (310.0, 160.8)
- added C41: 100n, decoup cap:CAPC2012X70, F.Cu at (9.91, 156.1)
- added C42: 100n, decoup cap:CAPC2012X70, F.Cu at (59.9, 175.1)
- added C43: 100n, decoup cap:CAPC2012X70, F.Cu at (125.6, 182.1)
- added C44: 100n, decoup cap:CAPC2012X70, F.Cu at (229.0, 175.0)
- added C45: 100n, decoup cap:CAPC2012X70, F.Cu at (290.7, 180.1)
- added C46: 100n, decoup cap:CAPC2012X70, F.Cu at (10.0, 174.9)
- added C47: 100n, decoup cap:CAPC2012X70, F.Cu at (328.9, 179.5)
- added C5: 100n, decoup cap:CAPC2012X70, F.Cu at (157.5, 74.3)
- added C6: 100n, decoup cap:CAPC2012X70, F.Cu at (195.6, 73.9)
- added C7: 100n, decoup cap:CAPC2012X70, F.Cu at (238.4, 74.8)
- added C8: 100n, decoup cap:CAPC2012X70, F.Cu at (276.5, 75.1)
- added C9: 100n, decoup cap:CAPC2012X70, F.Cu at (33.7, 75.1)
- added D87: D_Small, Diode_THT:D_DO-35_SOD27_P5.08mm_Vertical_KathodeUp, F.Cu at (233.4, 50.8)
- added MT_PCB_CD: MountingHole_2.2mm_M2_Pad, MountingHole:MountingHole_2.2mm_M2_Pad, F.Cu at (165.9, 181.0)
- added MT_PCB_CT: MountingHole_2.2mm_M2_Pad, MountingHole:MountingHole_2.2mm_M2_Pad, F.Cu at (165.9, 91.3)
- added MT_PCB_LD: MountingHole_2.2mm_M2_Pad, MountingHole:MountingHole_2.2mm_M2_Pad, F.Cu at (13.5, 181.0)
- added MT_PCB_LT: MountingHole_2.2mm_M2_Pad, MountingHole:MountingHole_2.2mm_M2_Pad, F.Cu at (15.1, 96.8)
- added MT_PCB_RD: MountingHole_2.2mm_M2_Pad, MountingHole:MountingHole_2.2mm_M2_Pad, F.Cu at (311.1, 181.0)
- added MT_PCB_RT: MountingHole_2.2mm_M2_Pad, MountingHole:MountingHole_2.2mm_M2_Pad, F.Cu at (311.1, 96.8)
- added MT_PLATE_CD: MountingHole_2.2mm_M2_Pad, MountingHole:MountingHole_2.2mm_M2_Pad, F.Cu at (165.9, 66.7)
- added MT_PLATE_CT: MountingHole_2.2mm_M2_Pad, MountingHole:MountingHole_2.2mm_M2_Pad, F.Cu at (165.9, 40.5)
- added MT_PLATE_LD: MountingHole_2.2mm_M2_Pad, MountingHole:MountingHole_2.2mm_M2_Pad, F.Cu at (-3.97, 66.7)
- added MT_PLATE_LT: MountingHole_2.2mm_M2_Pad, MountingHole:MountingHole_2.2mm_M2_Pad, F.Cu at (-3.97, 40.5)
- added MT_PLATE_RD: MountingHole_2.2mm_M2_Pad, MountingHole:MountingHole_2.2mm_M2_Pad, F.Cu at (331.0, 66.7)
- added MT_PLATE_RT: MountingHole_2.2mm_M2_Pad, MountingHole:MountingHole_2.2mm_M2_Pad, F.Cu at (331.0, 40.5)
Connections:
- ENC1 pad C: +5V -> GND
- ENC1 pad S1: VCC -> COL4
- ENC1 pad S2: ENC_SW -> ENC_S2
- WS76 pad 2: Net-(WS76-Pad2) -> D_ROW6
- WS77 pad 2: D_ROW6 -> Net-(WS77-Pad2)
- WS77 pad 4: Net-(WS76-Pad2) -> D_ROW6
- WS78 pad 4: D_ROW6 -> Net-(WS77-Pad2)
- WS83 pad 4: Net-(WS83-Pad4) -> Net-(WS82-Pad2)
- WS87 pad 2: Net-(WS83-Pad4) -> Net-(WS87-Pad2)
- WS87 pad 4: Net-(WS82-Pad2) -> Net-(WS86-Pad2)
Routing:
- net GND: track 0.00 -> 2618.9 mm, vias 0 -> 2
- net +5V: track 0.00 -> 2272.5 mm, vias 0 -> 5
- net COL0: track 0.00 -> 473.4 mm
- net COL4: track 0.00 -> 461.7 mm, vias 0 -> 1
- net COL1: track 0.00 -> 431.2 mm, vias 0 -> 3
- net COL2: track 0.00 -> 410.3 mm, vias 0 -> 1
- net COL3: track 0.00 -> 390.1 mm, vias 0 -> 1
- net D_ROW6: track 0.00 -> 373.1 mm
- net VCC: track 0.00 -> 359.6 mm, vias 0 -> 1
- net D_ROW5: track 0.00 -> 349.9 mm, vias 0 -> 2
- net ROW1: track 0.00 -> 349.2 mm
- net ROW2: track 0.00 -> 348.7 mm, vias 0 -> 1
- net D_ROW4: track 0.00 -> 345.8 mm
- net D_ROW3: track 0.00 -> 344.1 mm, vias 0 -> 2
- net ROW3: track 0.00 -> 342.5 mm
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Other:
- outline, holes or cut-outs redrawn
- board text added: "- swiftrax - squeezeonein - Fe - Martin Z. - David T."
- board text added: "CZTKey Rev. 0"
- board text added: "Special Thanks to:"
- board text added: "by cztrollolcz"

Commit message: Hopefully final touches
Parts:
- removed C1, C2: 100n, Capacitor_SMD:C_0603_1608Metric
- removed C10, C11, C12, C13, C14, C15, C16, C17, C18, C19, C20, C21, C22, C23, C24, C25, C26, C27, C28, C29, C3, C30, C31, C32, C33, C34, C35, C36, C37, C38, C39, C4, C40, C41, C42, C43, C44, C45, C46, C47, C5, C6, C7, C8, C9: 100n, decoup cap:CAPC2012X70
- removed MT_PCB_CD, MT_PCB_CT, MT_PCB_LD, MT_PCB_LT, MT_PCB_RD, MT_PCB_RT, MT_PLATE_CD, MT_PLATE_CT, MT_PLATE_LD, MT_PLATE_LT, MT_PLATE_RD, MT_PLATE_RT: MountingHole_2.2mm_M2_Pad, MountingHole:MountingHole_2.2mm_M2_Pad
- removed R2: 10k, Resistor_SMD:R_Array_Convex_4x0603
- removed R3, R4: 10K, Resistor_SMD:R_Array_Convex_4x0603
- removed WS1, WS10, WS11, WS12, WS13, WS14, WS15, WS16, WS17, WS18, WS19, WS2, WS20, WS21, WS22, WS23, WS24, WS25, WS26, WS27, WS28, WS29, WS3, WS30, WS31, WS32, WS33, WS34, WS35, WS36, WS37, WS38, WS39, WS4, WS40, WS41, WS42, WS43, WS44, WS45, WS46, WS47, WS48, WS49, WS5, WS50, WS51, WS52, WS53, WS54, WS55, WS56, WS57, WS58, WS59, WS6, WS60, WS61, WS62, WS63, WS64, WS65, WS66, WS67, WS68, WS69, WS7, WS70, WS71, WS72, WS73, WS74, WS75, WS76, WS77, WS78, WS79, WS8, WS80, WS81, WS82, WS83, WS84, WS85, WS86, WS87, WS9: WS2812B, WS2812B-edited:Neopixel_easy_LED_WS2812B_PLCC4_5.0x5.0mm_P3.2mm
- added BJ_LED5V1: Barrel_Jack_Switch, rgb led reverse mount:BarrelJackP1, F.Cu at (3.97, 26.9)
- added DC1: 100n, Capacitor_SMD:C_0805_2012Metric_Pad1.15x1.40mm_HandSolder, F.Cu at (33.7, 75.8)
- added DC10: 100n, Capacitor_SMD:C_0805_2012Metric_Pad1.15x1.40mm_HandSolder, F.Cu at (219.6, 75.8)
- added DC11: 100n, Capacitor_SMD:C_0805_2012Metric_Pad1.15x1.40mm_HandSolder, F.Cu at (238.6, 75.8)
- added DC12: 100n, Capacitor_SMD:C_0805_2012Metric_Pad1.15x1.40mm_HandSolder, F.Cu at (257.6, 75.8)
- added DC13: 100n, Capacitor_SMD:C_0805_2012Metric_Pad1.15x1.40mm_HandSolder, F.Cu at (276.6, 75.8)
- added DC14: 100n, Capacitor_SMD:C_0805_2012Metric_Pad1.15x1.40mm_HandSolder, F.Cu at (300.4, 75.8)
- added DC15: 100n, Capacitor_SMD:C_0805_2012Metric_Pad1.15x1.40mm_HandSolder, F.Cu at (33.7, 99.6)
- added DC16: 100n, Capacitor_SMD:C_0805_2012Metric_Pad1.15x1.40mm_HandSolder, F.Cu at (52.7, 99.6)
- added DC17: 100n, Capacitor_SMD:C_0805_2012Metric_Pad1.15x1.40mm_HandSolder, F.Cu at (71.8, 99.6)
- added DC18: 100n, Capacitor_SMD:C_0805_2012Metric_Pad1.15x1.40mm_HandSolder, F.Cu at (90.8, 99.6)
- added DC19: 100n, Capacitor_SMD:C_0805_2012Metric_Pad1.15x1.40mm_HandSolder, F.Cu at (109.9, 99.6)
- added DC2: 100n, Capacitor_SMD:C_0805_2012Metric_Pad1.15x1.40mm_HandSolder, F.Cu at (57.5, 75.8)
- added DC20: 100n, Capacitor_SMD:C_0805_2012Metric_Pad1.15x1.40mm_HandSolder, F.Cu at (128.9, 99.6)
- added DC21: 100n, Capacitor_SMD:C_0805_2012Metric_Pad1.15x1.40mm_HandSolder, F.Cu at (148.0, 99.6)
- added DC22: 100n, Capacitor_SMD:C_0805_2012Metric_Pad1.15x1.40mm_HandSolder, F.Cu at (167.0, 99.6)
- added DC23: 100n, Capacitor_SMD:C_0805_2012Metric_Pad1.15x1.40mm_HandSolder, F.Cu at (186.1, 99.6)
- added DC24: 100n, Capacitor_SMD:C_0805_2012Metric_Pad1.15x1.40mm_HandSolder, F.Cu at (205.1, 99.6)
- added DC25: 100n, Capacitor_SMD:C_0805_2012Metric_Pad1.15x1.40mm_HandSolder, F.Cu at (224.2, 99.6)
- added DC26: 100n, Capacitor_SMD:C_0805_2012Metric_Pad1.15x1.40mm_HandSolder, F.Cu at (243.2, 99.6)
- added DC27: 100n, Capacitor_SMD:C_0805_2012Metric_Pad1.15x1.40mm_HandSolder, F.Cu at (262.3, 99.6)
- added DC28: 100n, Capacitor_SMD:C_0805_2012Metric_Pad1.15x1.40mm_HandSolder, F.Cu at (288.8, 96.6)
- added DC29: 100n, Capacitor_SMD:C_0805_2012Metric_Pad1.15x1.40mm_HandSolder, F.Cu at (333.6, 99.6)
- added DC3: 100n, Capacitor_SMD:C_0805_2012Metric_Pad1.15x1.40mm_HandSolder, F.Cu at (76.6, 75.8)
- added DC30: 100n, Capacitor_SMD:C_0805_2012Metric_Pad1.15x1.40mm_HandSolder, F.Cu at (9.91, 99.6)
- added DC31: 100n, Capacitor_SMD:C_0805_2012Metric_Pad1.15x1.40mm_HandSolder, F.Cu at (39.4, 118.6)
- added DC32: 100n, Capacitor_SMD:C_0805_2012Metric_Pad1.15x1.40mm_HandSolder, F.Cu at (62.2, 118.6)
- added DC33: 100n, Capacitor_SMD:C_0805_2012Metric_Pad1.15x1.40mm_HandSolder, F.Cu at (81.3, 118.6)
- added DC34: 100n, Capacitor_SMD:C_0805_2012Metric_Pad1.15x1.40mm_HandSolder, F.Cu at (100.3, 118.6)
- added DC35: 100n, Capacitor_SMD:C_0805_2012Metric_Pad1.15x1.40mm_HandSolder, F.Cu at (119.4, 118.6)
- added DC36: 100n, Capacitor_SMD:C_0805_2012Metric_Pad1.15x1.40mm_HandSolder, F.Cu at (138.4, 118.6)
- added DC37: 100n, Capacitor_SMD:C_0805_2012Metric_Pad1.15x1.40mm_HandSolder, F.Cu at (157.5, 118.6)
- added DC38: 100n, Capacitor_SMD:C_0805_2012Metric_Pad1.15x1.40mm_HandSolder, F.Cu at (176.5, 118.6)
- added DC39: 100n, Capacitor_SMD:C_0805_2012Metric_Pad1.15x1.40mm_HandSolder, F.Cu at (195.6, 118.6)
- added DC4: 100n, Capacitor_SMD:C_0805_2012Metric_Pad1.15x1.40mm_HandSolder, F.Cu at (95.6, 75.8)
- added DC40: 100n, Capacitor_SMD:C_0805_2012Metric_Pad1.15x1.40mm_HandSolder, F.Cu at (214.6, 118.6)
- added DC41: 100n, Capacitor_SMD:C_0805_2012Metric_Pad1.15x1.40mm_HandSolder, F.Cu at (233.7, 118.6)
- added DC42: 100n, Capacitor_SMD:C_0805_2012Metric_Pad1.15x1.40mm_HandSolder, F.Cu at (252.7, 118.6)
- added DC43: 100n, Capacitor_SMD:C_0805_2012Metric_Pad1.15x1.40mm_HandSolder, F.Cu at (271.8, 118.6)
- added DC44: 100n, Capacitor_SMD:C_0805_2012Metric_Pad1.15x1.40mm_HandSolder, F.Cu at (295.7, 118.6)
- added DC45: 100n, Capacitor_SMD:C_0805_2012Metric_Pad1.15x1.40mm_HandSolder, F.Cu at (333.6, 118.6)
- added DC46: 100n, Capacitor_SMD:C_0805_2012Metric_Pad1.15x1.40mm_HandSolder, F.Cu at (9.91, 118.6)
- added DC47: 100n, Capacitor_SMD:C_0805_2012Metric_Pad1.15x1.40mm_HandSolder, F.Cu at (42.0, 137.7)
- added DC48: 100n, Capacitor_SMD:C_0805_2012Metric_Pad1.15x1.40mm_HandSolder, F.Cu at (67.1, 137.7)
- added DC49: 100n, Capacitor_SMD:C_0805_2012Metric_Pad1.15x1.40mm_HandSolder, F.Cu at (86.1, 137.7)
- added DC5: 100n, Capacitor_SMD:C_0805_2012Metric_Pad1.15x1.40mm_HandSolder, F.Cu at (114.7, 75.7)
- added DC50: 100n, Capacitor_SMD:C_0805_2012Metric_Pad1.15x1.40mm_HandSolder, F.Cu at (105.2, 137.7)
- added DC51: 100n, Capacitor_SMD:C_0805_2012Metric_Pad1.15x1.40mm_HandSolder, F.Cu at (124.2, 137.7)
- added DC52: 100n, Capacitor_SMD:C_0805_2012Metric_Pad1.15x1.40mm_HandSolder, F.Cu at (143.3, 137.7)
- added DC53: 100n, Capacitor_SMD:C_0805_2012Metric_Pad1.15x1.40mm_HandSolder, F.Cu at (162.3, 137.7)
- added DC54: 100n, Capacitor_SMD:C_0805_2012Metric_Pad1.15x1.40mm_HandSolder, F.Cu at (181.4, 137.7)
- added DC55: 100n, Capacitor_SMD:C_0805_2012Metric_Pad1.15x1.40mm_HandSolder, F.Cu at (200.4, 137.7)
- added DC56: 100n, Capacitor_SMD:C_0805_2012Metric_Pad1.15x1.40mm_HandSolder, F.Cu at (219.5, 137.7)
- added DC57: 100n, Capacitor_SMD:C_0805_2012Metric_Pad1.15x1.40mm_HandSolder, F.Cu at (238.5, 137.7)
- added DC58: 100n, Capacitor_SMD:C_0805_2012Metric_Pad1.15x1.40mm_HandSolder, F.Cu at (257.6, 137.7)
- added DC59: 100n, Capacitor_SMD:C_0805_2012Metric_Pad1.15x1.40mm_HandSolder, F.Cu at (286.6, 134.6)
- added DC6: 100n, Capacitor_SMD:C_0805_2012Metric_Pad1.15x1.40mm_HandSolder, F.Cu at (138.4, 75.9)
- added DC60: 100n, Capacitor_SMD:C_0805_2012Metric_Pad1.15x1.40mm_HandSolder, F.Cu at (333.6, 137.7)
- added DC61: 100n, Capacitor_SMD:C_0805_2012Metric_Pad1.15x1.40mm_HandSolder, F.Cu at (9.91, 137.7)
- added DC62: 100n, Capacitor_SMD:C_0805_2012Metric_Pad1.15x1.40mm_HandSolder, F.Cu at (43.7, 153.5)
- added DC63: 100n, Capacitor_SMD:C_0805_2012Metric_Pad1.15x1.40mm_HandSolder, F.Cu at (76.6, 156.7)
- added DC64: 100n, Capacitor_SMD:C_0805_2012Metric_Pad1.15x1.40mm_HandSolder, F.Cu at (95.6, 156.7)
- added DC65: 100n, Capacitor_SMD:C_0805_2012Metric_Pad1.15x1.40mm_HandSolder, F.Cu at (114.7, 156.7)
- added DC66: 100n, Capacitor_SMD:C_0805_2012Metric_Pad1.15x1.40mm_HandSolder, F.Cu at (133.7, 156.7)
- added DC67: 100n, Capacitor_SMD:C_0805_2012Metric_Pad1.15x1.40mm_HandSolder, F.Cu at (152.8, 156.7)
- added DC68: 100n, Capacitor_SMD:C_0805_2012Metric_Pad1.15x1.40mm_HandSolder, F.Cu at (171.8, 156.7)
- added DC69: 100n, Capacitor_SMD:C_0805_2012Metric_Pad1.15x1.40mm_HandSolder, F.Cu at (190.9, 156.7)
- added DC7: 100n, Capacitor_SMD:C_0805_2012Metric_Pad1.15x1.40mm_HandSolder, F.Cu at (157.5, 75.8)
- added DC70: 100n, Capacitor_SMD:C_0805_2012Metric_Pad1.15x1.40mm_HandSolder, F.Cu at (209.9, 156.7)
- added DC71: 100n, Capacitor_SMD:C_0805_2012Metric_Pad1.15x1.40mm_HandSolder, F.Cu at (229.0, 156.7)
- added DC72: 100n, Capacitor_SMD:C_0805_2012Metric_Pad1.15x1.40mm_HandSolder, F.Cu at (248.0, 156.7)
- added DC73: 100n, Capacitor_SMD:C_0805_2012Metric_Pad1.15x1.40mm_HandSolder, F.Cu at (275.3, 156.7)
- added DC74: 100n, Capacitor_SMD:C_0805_2012Metric_Pad1.15x1.40mm_HandSolder, F.Cu at (309.9, 156.7)
- added DC75: 100n, Capacitor_SMD:C_0805_2012Metric_Pad1.15x1.40mm_HandSolder, F.Cu at (333.6, 156.7)
- added DC76: 100n, Capacitor_SMD:C_0805_2012Metric_Pad1.15x1.40mm_HandSolder, F.Cu at (9.91, 156.7)
- added DC78: 100n, Capacitor_SMD:C_0805_2012Metric_Pad1.15x1.40mm_HandSolder, F.Cu at (9.91, 175.8)
- added DC79: 100n, Capacitor_SMD:C_0805_2012Metric_Pad1.15x1.40mm_HandSolder, F.Cu at (37.2, 175.8)
- added DC8: 100n, Capacitor_SMD:C_0805_2012Metric_Pad1.15x1.40mm_HandSolder, F.Cu at (176.5, 75.8)
- added DC80: 100n, Capacitor_SMD:C_0805_2012Metric_Pad1.15x1.40mm_HandSolder, F.Cu at (61.0, 175.8)
- added DC81: 100n, Capacitor_SMD:C_0805_2012Metric_Pad1.15x1.40mm_HandSolder, F.Cu at (84.8, 175.8)
- added DC82: 100n, Capacitor_SMD:C_0805_2012Metric_Pad1.15x1.40mm_HandSolder, F.Cu at (156.2, 177.2)
- added DC83: 100n, Capacitor_SMD:C_0805_2012Metric_Pad1.15x1.40mm_HandSolder, F.Cu at (230.1, 175.8)
- added DC84: 100n, Capacitor_SMD:C_0805_2012Metric_Pad1.15x1.40mm_HandSolder, F.Cu at (258.7, 175.8)
- added DC85: 100n, Capacitor_SMD:C_0805_2012Metric_Pad1.15x1.40mm_HandSolder, F.Cu at (290.8, 175.8)
- added DC86: 100n, Capacitor_SMD:C_0805_2012Metric_Pad1.15x1.40mm_HandSolder, F.Cu at (309.9, 175.8)
- added DC87: 100n, Capacitor_SMD:C_0805_2012Metric_Pad1.15x1.40mm_HandSolder, F.Cu at (328.8, 175.8)
- added DC9: 100n, Capacitor_SMD:C_0805_2012Metric_Pad1.15x1.40mm_HandSolder, F.Cu at (195.6, 75.8)
- added EXT_IC1: 74LVC1G17GV,125, SamacSys_Parts:SOT95P275X110-5N, F.Cu at (15.9, 69.5)
- added LED1: YS-SK6812MINI-E, rgb led reverse mount:SK6812MINIE-simple, F.Cu at (25.4, 75.4)
- added LED10: YS-SK6812MINI-E, rgb led reverse mount:SK6812MINIE-simple, F.Cu at (211.1, 75.4)
- added LED11: YS-SK6812MINI-E, rgb led reverse mount:SK6812MINIE-simple, F.Cu at (230.2, 75.4)
- added LED12: YS-SK6812MINI-E, rgb led reverse mount:SK6812MINIE-simple, F.Cu at (249.2, 75.4)
- added LED13: YS-SK6812MINI-E, rgb led reverse mount:SK6812MINIE-simple, F.Cu at (268.3, 75.4)
- added LED14: YS-SK6812MINI-E, rgb led reverse mount:SK6812MINIE-simple, F.Cu at (292.1, 75.4)
- added LED15: YS-SK6812MINI-E, rgb led reverse mount:SK6812MINIE-simple, F.Cu at (1.59, 99.2)
- added LED16: YS-SK6812MINI-E, rgb led reverse mount:SK6812MINIE-simple, F.Cu at (25.4, 99.2)
- added LED17: YS-SK6812MINI-E, rgb led reverse mount:SK6812MINIE-simple, F.Cu at (44.5, 99.2)
- added LED18: YS-SK6812MINI-E, rgb led reverse mount:SK6812MINIE-simple, F.Cu at (63.5, 99.2)
- added LED19: YS-SK6812MINI-E, rgb led reverse mount:SK6812MINIE-simple, F.Cu at (82.5, 99.2)
- added LED2: YS-SK6812MINI-E, rgb led reverse mount:SK6812MINIE-simple, F.Cu at (49.2, 75.4)
- added LED20: YS-SK6812MINI-E, rgb led reverse mount:SK6812MINIE-simple, F.Cu at (101.6, 99.2)
- added LED21: YS-SK6812MINI-E, rgb led reverse mount:SK6812MINIE-simple, F.Cu at (120.7, 99.2)
- added LED22: YS-SK6812MINI-E, rgb led reverse mount:SK6812MINIE-simple, F.Cu at (139.7, 99.2)
- added LED23: YS-SK6812MINI-E, rgb led reverse mount:SK6812MINIE-simple, F.Cu at (158.8, 99.2)
- added LED24: YS-SK6812MINI-E, rgb led reverse mount:SK6812MINIE-simple, F.Cu at (177.8, 99.2)
- added LED25: YS-SK6812MINI-E, rgb led reverse mount:SK6812MINIE-simple, F.Cu at (196.8, 99.2)
- added LED26: YS-SK6812MINI-E, rgb led reverse mount:SK6812MINIE-simple, F.Cu at (215.9, 99.2)
- added LED27: YS-SK6812MINI-E, rgb led reverse mount:SK6812MINIE-simple, F.Cu at (234.9, 99.2)
- added LED28: YS-SK6812MINI-E, rgb led reverse mount:SK6812MINIE-simple, F.Cu at (254.0, 99.2)
- added LED29: YS-SK6812MINI-E, rgb led reverse mount:SK6812MINIE-simple, F.Cu at (282.6, 99.2)
- added LED3: YS-SK6812MINI-E, rgb led reverse mount:SK6812MINIE-simple, F.Cu at (68.3, 75.4)
- added LED30: YS-SK6812MINI-E, rgb led reverse mount:SK6812MINIE-simple, F.Cu at (325.4, 99.2)
- added LED31: YS-SK6812MINI-E, rgb led reverse mount:SK6812MINIE-simple, F.Cu at (1.59, 118.3)
- added LED32: YS-SK6812MINI-E, rgb led reverse mount:SK6812MINIE-simple, F.Cu at (30.2, 118.3)
- added LED33: YS-SK6812MINI-E, rgb led reverse mount:SK6812MINIE-simple, F.Cu at (54.0, 118.3)
- added LED34: YS-SK6812MINI-E, rgb led reverse mount:SK6812MINIE-simple, F.Cu at (73.0, 118.3)
- added LED35: YS-SK6812MINI-E, rgb led reverse mount:SK6812MINIE-simple, F.Cu at (92.1, 118.3)
- added LED36: YS-SK6812MINI-E, rgb led reverse mount:SK6812MINIE-simple, F.Cu at (111.1, 118.3)
- added LED37: YS-SK6812MINI-E, rgb led reverse mount:SK6812MINIE-simple, F.Cu at (130.2, 118.3)
- added LED38: YS-SK6812MINI-E, rgb led reverse mount:SK6812MINIE-simple, F.Cu at (149.2, 118.3)
- added LED39: YS-SK6812MINI-E, rgb led reverse mount:SK6812MINIE-simple, F.Cu at (168.3, 118.3)
- added LED4: YS-SK6812MINI-E, rgb led reverse mount:SK6812MINIE-simple, F.Cu at (87.3, 75.4)
- added LED40: YS-SK6812MINI-E, rgb led reverse mount:SK6812MINIE-simple, F.Cu at (187.3, 118.3)
- added LED41: YS-SK6812MINI-E, rgb led reverse mount:SK6812MINIE-simple, F.Cu at (206.4, 118.3)
- added LED42: YS-SK6812MINI-E, rgb led reverse mount:SK6812MINIE-simple, F.Cu at (225.4, 118.3)
- added LED43: YS-SK6812MINI-E, rgb led reverse mount:SK6812MINIE-simple, F.Cu at (244.5, 118.3)
- added LED44: YS-SK6812MINI-E, rgb led reverse mount:SK6812MINIE-simple, F.Cu at (263.5, 118.3)
- added LED45: YS-SK6812MINI-E, rgb led reverse mount:SK6812MINIE-simple, F.Cu at (287.3, 118.3)
- added LED46: YS-SK6812MINI-E, rgb led reverse mount:SK6812MINIE-simple, F.Cu at (325.4, 118.3)
- added LED47: YS-SK6812MINI-E, rgb led reverse mount:SK6812MINIE-simple, F.Cu at (1.59, 137.3)
- added LED48: YS-SK6812MINI-E, rgb led reverse mount:SK6812MINIE-simple, F.Cu at (32.5, 137.3)
- added LED49: YS-SK6812MINI-E, rgb led reverse mount:SK6812MINIE-simple, F.Cu at (58.7, 137.3)
- added LED5: YS-SK6812MINI-E, rgb led reverse mount:SK6812MINIE-simple, F.Cu at (106.4, 75.4)
- added LED50: YS-SK6812MINI-E, rgb led reverse mount:SK6812MINIE-simple, F.Cu at (77.8, 137.3)
- added LED51: YS-SK6812MINI-E, rgb led reverse mount:SK6812MINIE-simple, F.Cu at (96.8, 137.3)
- added LED52: YS-SK6812MINI-E, rgb led reverse mount:SK6812MINIE-simple, F.Cu at (115.9, 137.3)
- added LED53: YS-SK6812MINI-E, rgb led reverse mount:SK6812MINIE-simple, F.Cu at (134.9, 137.3)
- added LED54: YS-SK6812MINI-E, rgb led reverse mount:SK6812MINIE-simple, F.Cu at (154.0, 137.3)
- added LED55: YS-SK6812MINI-E, rgb led reverse mount:SK6812MINIE-simple, F.Cu at (173.0, 137.3)
- added LED56: YS-SK6812MINI-E, rgb led reverse mount:SK6812MINIE-simple, F.Cu at (192.1, 137.3)
- added LED57: YS-SK6812MINI-E, rgb led reverse mount:SK6812MINIE-simple, F.Cu at (211.1, 137.3)
- added LED58: YS-SK6812MINI-E, rgb led reverse mount:SK6812MINIE-simple, F.Cu at (230.2, 137.3)
- added LED59: YS-SK6812MINI-E, rgb led reverse mount:SK6812MINIE-simple, F.Cu at (249.2, 137.3)
- added LED6: YS-SK6812MINI-E, rgb led reverse mount:SK6812MINIE-simple, F.Cu at (130.2, 75.4)
- added LED60: YS-SK6812MINI-E, rgb led reverse mount:SK6812MINIE-simple, F.Cu at (280.2, 137.3)
- added LED61: YS-SK6812MINI-E, rgb led reverse mount:SK6812MINIE-simple, F.Cu at (325.4, 137.3)
- added LED62: YS-SK6812MINI-E, rgb led reverse mount:SK6812MINIE-simple, F.Cu at (1.59, 156.4)
- added LED63: YS-SK6812MINI-E, rgb led reverse mount:SK6812MINIE-simple, F.Cu at (37.3, 156.4)
- added LED64: YS-SK6812MINI-E, rgb led reverse mount:SK6812MINIE-simple, F.Cu at (68.3, 156.4)
- added LED65: YS-SK6812MINI-E, rgb led reverse mount:SK6812MINIE-simple, F.Cu at (87.3, 156.4)
- added LED66: YS-SK6812MINI-E, rgb led reverse mount:SK6812MINIE-simple, F.Cu at (106.4, 156.4)
- added LED67: YS-SK6812MINI-E, rgb led reverse mount:SK6812MINIE-simple, F.Cu at (125.4, 156.4)
- added LED68: YS-SK6812MINI-E, rgb led reverse mount:SK6812MINIE-simple, F.Cu at (144.5, 156.4)
- added LED69: YS-SK6812MINI-E, rgb led reverse mount:SK6812MINIE-simple, F.Cu at (163.5, 156.4)
- added LED7: YS-SK6812MINI-E, rgb led reverse mount:SK6812MINIE-simple, F.Cu at (149.2, 75.4)
- added LED70: YS-SK6812MINI-E, rgb led reverse mount:SK6812MINIE-simple, F.Cu at (182.6, 156.4)
- added LED71: YS-SK6812MINI-E, rgb led reverse mount:SK6812MINIE-simple, F.Cu at (201.6, 156.4)
- added LED72: YS-SK6812MINI-E, rgb led reverse mount:SK6812MINIE-simple, F.Cu at (220.7, 156.4)
- added LED73: YS-SK6812MINI-E, rgb led reverse mount:SK6812MINIE-simple, F.Cu at (239.7, 156.4)
- added LED74: YS-SK6812MINI-E, rgb led reverse mount:SK6812MINIE-simple, F.Cu at (265.9, 156.4)
- added LED75: YS-SK6812MINI-E, rgb led reverse mount:SK6812MINIE-simple, F.Cu at (301.6, 156.4)
- added LED76: YS-SK6812MINI-E, rgb led reverse mount:SK6812MINIE-simple, F.Cu at (326.2, 156.4)
- added LED78: YS-SK6812MINI-E, rgb led reverse mount:SK6812MINIE-simple, F.Cu at (1.59, 175.4)
- added LED79: YS-SK6812MINI-E, rgb led reverse mount:SK6812MINIE-simple, F.Cu at (27.8, 175.4)
- added LED8: YS-SK6812MINI-E, rgb led reverse mount:SK6812MINIE-simple, F.Cu at (168.3, 75.4)
- added LED80: YS-SK6812MINI-E, rgb led reverse mount:SK6812MINIE-simple, F.Cu at (51.6, 175.4)
- added LED81: YS-SK6812MINI-E, rgb led reverse mount:SK6812MINIE-simple, F.Cu at (75.4, 175.4)
- added LED82: YS-SK6812MINI-E, rgb led reverse mount:SK6812MINIE-simple, F.Cu at (146.8, 175.4)
- added LED83: YS-SK6812MINI-E, rgb led reverse mount:SK6812MINIE-simple, F.Cu at (220.7, 175.4)
- added LED84: YS-SK6812MINI-E, rgb led reverse mount:SK6812MINIE-simple, F.Cu at (249.2, 175.4)
- added LED85: YS-SK6812MINI-E, rgb led reverse mount:SK6812MINIE-simple, F.Cu at (282.6, 175.4)
- added LED86: YS-SK6812MINI-E, rgb led reverse mount:SK6812MINIE-simple, F.Cu at (301.6, 175.4)
- added LED87: YS-SK6812MINI-E, rgb led reverse mount:SK6812MINIE-simple, F.Cu at (320.7, 175.4)
- added LED9: YS-SK6812MINI-E, rgb led reverse mount:SK6812MINIE-simple, F.Cu at (187.3, 75.4)
- added PCB_BC1: MountingHole_Pad, MountingHole:MountingHole_2.2mm_M2_Pad, F.Cu at (172.2, 181.0)
- added PCB_BL1: MountingHole_Pad, MountingHole:MountingHole_2.2mm_M2_Pad, F.Cu at (13.5, 181.0)
- added PCB_BR1: MountingHole_Pad, MountingHole:MountingHole_2.2mm_M2_Pad, F.Cu at (330.2, 181.8)
- added PCB_MC1: MountingHole_Pad, MountingHole:MountingHole_2.2mm_M2_Pad, F.Cu at (158.8, 131.8)
- added PCB_TC1: MountingHole_Pad, MountingHole:MountingHole_2.2mm_M2_Pad, F.Cu at (172.2, 92.9)
- added PCB_TL1: MountingHole_Pad, MountingHole:MountingHole_2.2mm_M2_Pad, F.Cu at (2.38, 92.9)
- added PCB_TR1: MountingHole_Pad, MountingHole:MountingHole_2.2mm_M2_Pad, F.Cu at (330.2, 77.8)
- added PLATE_BC1: MountingHole_Pad, MountingHole:MountingHole_2.2mm_M2_Pad, F.Cu at (172.2, 67.5)
- added PLATE_BL1: MountingHole_Pad, MountingHole:MountingHole_2.2mm_M2_Pad, F.Cu at (-3.17, 64.3)
- added PLATE_BR1: MountingHole_Pad, MountingHole:MountingHole_2.2mm_M2_Pad, F.Cu at (330.2, 64.3)
- added PLATE_TC1: MountingHole_Pad, MountingHole:MountingHole_2.2mm_M2_Pad, F.Cu at (169.9, 20.6)
- added PLATE_TL1: MountingHole_Pad, MountingHole:MountingHole_2.2mm_M2_Pad, F.Cu at (-3.17, 20.6)
- added PLATE_TR1: MountingHole_Pad, MountingHole:MountingHole_2.2mm_M2_Pad, F.Cu at (330.2, 20.6)
- R1: value 10k -> 300-500 - C422828; footprint Resistor_SMD:R_Array_Convex_4x0603 -> Resistor_SMD:R_0805_2012Metric_Pad1.15x1.40mm_HandSolder
- moved U1 296.7 mm to (19.1, 35.7), turned to 0 degrees
- moved D0 34.1 mm to (267.5, 50.8)
- moved D38 33.4 mm to (252.5, 44.5)
- moved D53 33.4 mm to (255.7, 44.5)
- moved D67 33.4 mm to (258.8, 44.5)
- moved D9 33.4 mm to (246.1, 44.5)
- moved D23 33.4 mm to (249.3, 44.5)
- moved D28 33.4 mm to (249.2, 57.1)
- moved D71 33.4 mm to (255.6, 57.1)
- moved D14 33.4 mm to (246.1, 57.1)
- moved D43 33.4 mm to (252.4, 57.1)
- moved D73 33.4 mm to (258.8, 57.1)
- moved D13 32.6 mm to (223.9, 44.5)
- moved D27 32.6 mm to (227.1, 44.5)
- moved D42 32.6 mm to (230.3, 44.5)
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- renumbered D87 to D0
Connections:
- net GND renamed EXT_GND
- D0 pad 1: ROW5 -> ROW0
- ENC1 pad A: Net-(ENC1-PadA) -> ENC_A
- ENC1 pad B: Net-(ENC1-PadB) -> ENC_B
- ENC1 pad S1: COL4 -> COL0
- OLED1 pad 2: VCC -> +5V
- R1 pad 1: VCC -> RGB_MATRIX
- R1 pad 2: Net-(ENC1-PadA) -> Net-(R1-Pad2)
- U1 pad B10: ENC_SW -> Net-(R1-Pad2)
Routing:
- net EXT_5V: track 0.00 -> 3043.8 mm, vias 0 -> 42
- net +5V: track 2272.5 -> 34.6 mm, vias 5 -> 0
- net EXT_GND: track 2618.9 -> 3302.6 mm, vias 2 -> 38
- net D_ROW6: track 373.1 -> 0.00 mm
- net VCC: track 359.6 -> 0.00 mm, vias 1 -> 0
- net D_ROW5: track 349.9 -> 0.00 mm, vias 2 -> 0
- net D_ROW4: track 345.8 -> 0.00 mm
- net D_ROW3: track 344.1 -> 0.00 mm, vias 2 -> 0
- net D_ROW2: track 313.2 -> 0.00 mm, vias 2 -> 0
- net COL13: track 189.5 -> 476.5 mm, vias 1 -> 3
- net ENC_B: track 311.5 -> 39.4 mm, vias 1 -> 0
- net COL0: track 473.4 -> 206.4 mm, vias 0 -> 1
- net COL14: track 136.8 -> 402.0 mm, vias 1 -> 0
- net COL15: track 158.8 -> 423.8 mm, vias 0 -> 2
- net ENC_A: track 304.3 -> 43.8 mm
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Other:
- board size 343 x 159 mm -> 342.9 x 174.6 mm
- board text added: "CZTKey"
- board text added: "Rev.0"
- board text removed: "- swiftrax - squeezeonein - Fe - Martin Z. - David T."
- board text removed: "CZTKey Rev. 0"
- board text removed: "Special Thanks to:"
