File: pcb/CZTKeyRev0.kicad_pcb (KiCad board)
At the start: 2 copper layers, 342.9 x 174.6 mm, 364 parts, among them U1 proton_c

Commit message: FR4 Plate and stuff
Parts:
- moved PLATE_BC1 2.86 mm to (170.7, 65.1)
Routing:
- net Net-(D24-Pad2): track 95.0 -> 98.6 mm
- net COL14: track 402.0 -> 404.1 mm
- net COL15: track 423.8 -> 425.2 mm
Other:
- board size 342.9 x 174.6 mm -> 342.9 x 177 mm
