File: pcb/CZTKeyRev0Plate.kicad_pcb (KiCad board)
At the start: 2 copper layers, 342.9 x 121.5 mm, 93 parts

Commit message: Plate Gerbers
Parts:
- removed MX_0, MX_1, MX_2, MX_3, MX_4, MX_5, MX_6, MX_7, MX_8, MX_9, MX_A1, MX_B1, MX_BR_L1, MX_BR_R1, MX_C1, MX_COMMA1, MX_D1, MX_DELETE1, MX_DOT1, MX_DOWN1, MX_E1, MX_EQUAL1, MX_ESC1, MX_F0, MX_F1, MX_F10, MX_F11, MX_F12, MX_F2, MX_F3, MX_F4, MX_F5, MX_F6, MX_F7, MX_F8, MX_F9, MX_G1, MX_H1, MX_I1, MX_INSERT1, MX_J1, MX_K1, MX_L1, MX_LEFT1, MX_M1, MX_MAC1, MX_MAC2, MX_MAC3, MX_MAC4, MX_MAC5, MX_MINUS1, MX_N1, MX_O1, MX_P1, MX_PGDWN1, MX_PGUP1, MX_PRTSC1, MX_Q1, MX_QUOTE1, MX_R1, MX_RIGHT1, MX_S1, MX_SEMIC1, MX_SLASH1, MX_T1, MX_TILDE1, MX_U1, MX_UP1, MX_V1, MX_W1, MX_X1, MX_Y1, MX_Z1: MX-NoLED, MX_Alps_Hybrid:MX-1U-NoLED
- removed MX_ALT_L1, MX_CTRL_L1, MX_WIN1: MX-NoLED, MX_Alps_Hybrid:MX-1.25U-NoLED
- removed MX_ALT_R1, MX_BCKSLASH1, MX_CTRL_R1, MX_TAB1: MX-NoLED, MX_Alps_Hybrid:MX-1.5U-NoLED
- removed MX_BACKSPACE1: MX-NoLED, MX_Alps_Hybrid:MX-2U-NoLED
- removed MX_CAPS1, MX_SHIFT_R1: MX-NoLED, MX_Alps_Hybrid:MX-1.75U-NoLED
- removed MX_ENTER1, MX_SHIFT_L1: MX-NoLED, MX_Alps_Hybrid:MX-2.25U-NoLED
- removed MX_SPACE1: MX-NoLED, MX_Alps_Hybrid:MX-6.25U-NoLED

Commit message: ????
Other:
- board size 342.9 x 121.5 mm -> 703.4 x 121.5 mm
